Commit message: Fix rounding error

File: src/muvu_description/urdf/muvu_circle_body.xacro (robot description, xacro)
@@ -3,10 +3,10 @@
   <!-- DEFINING GENERIC PROPERTIES THAT ARE USED IN THE XACRO FILE -->
   <!-- along x axis -->
-  <xacro:property name="base_length" value="0.5"/>
+  <xacro:property name="base_dia" value="0.5"/>
   <!-- along y axis -->
-  <xacro:property name="base_width" value="0.5"/>
+  <xacro:property name="base_dia" value="0.5"/>
   <!-- along z axis -->
-  <xacro:property name="base_height" value="0.1"/>
-  <xacro:property name="base_mass" value="10"/>
+  <xacro:property name="base_height" value="0.099"/>
+  <xacro:property name="base_mass" value="50"/>
   <xacro:property name="wheel_dia" value="0.1"/>
   <xacro:property name="wheel_height" value="0.05"/>
@@ -26,10 +26,10 @@
     <inertial>
       <mass value="${base_mass}" />
-      <inertia ixx="${(1/12)*base_mass*((base_width*base_width)+(base_height*base_height))}"
+      <inertia ixx="${(1/12)*base_mass*((base_dia*base_dia)+(base_height*base_height))}"
         ixy="0.0"
         ixz="0.0"
-        iyy="${(1/12)*base_mass*((base_height*base_height)+(base_length*base_length))}"
+        iyy="${(1/12)*base_mass*((base_height*base_height)+(base_dia*base_dia))}"
         iyz="0.0"
-        izz="${(1/12)*base_mass*((base_width*base_width)+(base_length*base_length))}" />
+        izz="${(1/12)*base_mass*((base_dia*base_dia)+(base_dia*base_dia))}" />
     </inertial>
   </xacro:macro>
@@ -41,6 +41,6 @@
   </xacro:macro>
   <!-- MACRO FOR GENERIC WHEEL. SUPPLY PARAMS TO PLACE THEM, JOINT INCLUDEDE IN MACRO -->
-  <xacro:macro name="wheel" params="left_right front_back relx rely">
-    <link name="${left_right}_${front_back}_wheel">
+  <xacro:macro name="wheel" params="left_right rely">
+    <link name="${left_right}_wheel">
       <visual>
         <origin xyz="0 0 0" rpy="${pi/2} 0 0"/>
@@ -58,9 +58,9 @@
       <xacro:wheel_inertial/>
     </link>
-    <joint name="${left_right}_${front_back}_wheel_to_base_link" type="continuous">
-      <origin xyz="${relx*((base_length/2)-wheel_dia/2)} ${rely*((base_width/2-wheel_height/2))} ${wheel_dia/2}" rpy="0 0 0"/>
+    <joint name="${left_right}_wheel_to_base_link" type="continuous">
+      <origin xyz="0 ${rely*((base_dia/2+wheel_height/2))} ${wheel_dia/2}" rpy="0 0 0"/>
       <axis xyz="0 1 0" rpy="0 0 0"/>
       <parent link="base_link"/>
-      <child link="${left_right}_${front_back}_wheel"/>
+      <child link="${left_right}_wheel"/>
     </joint>
   </xacro:macro>
@@ -70,14 +70,14 @@
   <link name="base_link">
     <visual>
-      <origin xyz="0 0 ${wheel_dia + base_height/2}" rpy="0 0 0"/>
+      <origin xyz="0 0 ${wheel_dia/2}" rpy="0 0 0"/>
       <geometry>
-        <box size="${base_length} ${base_width} ${base_height}"/>
+        <cylinder length="${base_height}" radius="${base_dia/2}"/>
       </geometry>
       <material name="white"/>
     </visual>
     <collision name="base_link_collision">
-      <origin xyz="0 0 ${wheel_dia + base_height/2}" rpy="0 0 0"/>
+      <origin xyz="0 0 ${wheel_dia/2}" rpy="0 0 0"/>
       <geometry>
-        <box size="${base_length} ${base_width} ${base_height}"/>
+        <cylinder length="${base_height}" radius="${base_dia/2}"/>
       </geometry>
     </collision>
@@ -90,8 +90,6 @@
   </joint>
   <!-- CREATING AN INSTANCE OF EACH WHEEL -->
-  <xacro:wheel left_right="left" front_back="front" relx="1" rely="1"/>
-  <xacro:wheel left_right="left" front_back="back" relx="-1" rely="1"/>
-  <xacro:wheel left_right="right" front_back="back" relx="-1" rely="-1"/>
-  <xacro:wheel left_right="right" front_back="front" relx="1" rely="-1"/>
+  <xacro:wheel left_right="left" rely="1"/>
+  <xacro:wheel left_right="right" rely="-1"/>
   <!--_______________________ Hokuyo Laser _______________________-->
   <link name="hokuyo_link">
@@ -117,5 +115,5 @@
   <joint name="hokuyo_joint" type="fixed">
     <axis xyz="0 1 0" />
-    <origin xyz="0 0 ${base_height+wheel_dia+0.025}" rpy="0 0 0"/>
+    <origin xyz="0 0 ${wheel_dia+0.025}" rpy="0 0 0"/>
     <parent link="base_link"/>
     <child link="hokuyo_link"/>
@@ -159,15 +157,14 @@
   <!-- SKID STEER PLUGIN -->
   <gazebo>
-    <plugin name="skid_steer_drive_controller" filename="libgazebo_ros_skid_steer_drive.so">
+    <plugin name="differential_drive_controller" filename="libgazebo_ros_diff_drive.so">
       <updateRate>100.0</updateRate>
       <robotNamespace>/muvu</robotNamespace>
-      <leftFrontJoint>left_front_wheel_to_base_link</leftFrontJoint>
-      <rightFrontJoint>right_front_wheel_to_base_link</rightFrontJoint>
-      <leftRearJoint>left_back_wheel_to_base_link</leftRearJoint>
-      <rightRearJoint>right_back_wheel_to_base_link</rightRearJoint>
+      <leftJoint>left_wheel_to_base_link</leftJoint>
+      <rightJoint>right_wheel_to_base_link</rightJoint>
       <wheelSeparation>0.5</wheelSeparation>
       <wheelDiameter>0.1</wheelDiameter>
+      <wheelAcceleration>1.0</wheelAcceleration>
+      <wheelTorque>5</wheelTorque>
       <robotBaseFrame>base_link</robotBaseFrame>
-      <torque>5</torque>
       <commandTopic>cmd_vel</commandTopic>
       <broadcastTF>false</broadcastTF>
@@ -177,6 +174,5 @@
   <gazebo>
     <plugin name="joint_state_publisher" filename="libgazebo_ros_joint_state_publisher.so">
-      <jointName>left_front_wheel_to_base_link, left_back_wheel_to_base_link,
-      right_front_wheel_to_base_link, right_back_wheel_to_base_link</jointName>
+      <jointName>left_wheel_to_base_link, right_wheel_to_base_link</jointName>
     </plugin>
   </gazebo>
